Commit message: Microban v2 model (Radxa): walking (default) and climbing-mode forearms / feet, CAD masses, IMU mount
src/model/mjcf/robot.xml (scene.xml) and robot_climb.xml (scene_climb.xml), urdf/robot.urdf and robot_climb.urdf
(kinematics, from the MJCFs): the same robot except the forearms and the feet (walking ones from the v1 model with their
collision primitives; ball hands and climbing feet). Servos sticking out as boxes, the trunk as four hulls, other parts
as convex pieces. Shoulder pitch zero turned to the code's convention (arm down; MOTOR_OFFSET on the robot). Same
joints, torque actuators (xl330) and IMU sensors as v1; IMU_MOUNT_QUAT follows the new imu site. The sim group pins
BAM to the commit with vin_drop_gain (sim/mujoco_controller.py). Docs: docs/model.md.

Co-Authored-By: Claude Opus 5.5 <noreply@anthropic.com>
Claude-Session: https://claude.ai/code/session_018d9UckeD9X4H8Nj272GbiR

File: src/model/urdf/robot.urdf (robot description, URDF)
Before this commit: robot urdf, 24 links, 23 joints
Links:
- link ankle_block__configuration_left: mass 0.04722 -> 0.048013
- link ankle_block__configuration_right: mass 0.04722 -> 0.048013
- link body: mass 1e-9 -> 1e-09
- link femur__configuration_left: mass 0.014726 -> 0.0161197
- link femur__configuration_right: mass 0.014726 -> 0.0161197
- link head: mass 0.0166215 -> 0.0169699
- link hip: mass 0.00884451 -> 0.00988978
- link hip_2: mass 0.00884451 -> 0.00988978
- link hip_block__configuration_left: mass 0.04763 -> 0.048423
- link hip_block__configuration_right: mass 0.04763 -> 0.048423
- link humerus__configuration_left: mass 0.0416867 -> 0.042744
- link humerus__configuration_right: mass 0.0416867 -> 0.042744
- link imu: mass 1e-9 -> 1e-09
- link left_foot: mass 1e-9 -> 1e-09
- link right_foot: mass 1e-9 -> 1e-09
- link shoulder: mass 0.00898451 -> 0.0100298
- link shoulder_2: mass 0.00898451 -> 0.0100298
- link tibia__configuration_left: mass 0.0300463 -> 0.0312719
- link tibia__configuration_right: mass 0.0300463 -> 0.0312719
- link trunk: mass 0.347283 -> 0.283162
Joints:
- joint body_frame: origin xyz=0 0 0 rpy=0 0 0 -> xyz=0 0 0 rpy=0 -0 0
- joint head: limit lower=-1.5708 upper=1.5708 effort=10 velocity=10 -> lower=-1.5708 upper=1.5708 effort=0.6 velocity=6.6; origin xyz=-0.00204165 -0 0.126 rpy=0 0 1.5708 -> xyz=0.00195835 0 0.126 rpy=0 -0 1.57079633
- joint imu_frame: origin xyz=0.01483 -0.002 0.0675 rpy=1.5708 -0 -1.5708 -> xyz=-0.01421 -0.015 0.044 rpy=1.57079633 -0 1.57079633
- joint left_ankle_pitch: limit lower=-1.5708 upper=0.610865 effort=10 velocity=10 -> lower=-1.5708 upper=0.610865 effort=0.6 velocity=6.6; origin xyz=-0.008 0.0612131 -0 rpy=-0 -0 3.14159 -> xyz=-0.008 0.0612131 0 rpy=0 0 3.14159265
- joint left_ankle_roll: limit lower=-0.610865 upper=0.610865 effort=10 velocity=10 -> lower=-0.610865 upper=0.610865 effort=0.6 velocity=6.6; origin xyz=0.0385 0 -0.0145 rpy=-0 -1.5708 0 -> xyz=0.0385 0 -0.0145 rpy=0 -1.57079633 0
- joint left_elbow: limit lower=-2.18166 upper=2.18166 effort=10 velocity=10 -> lower=-2.18166 upper=2.18166 effort=0.6 velocity=6.6; origin xyz=-0.0145 0.0515 -0.0145 rpy=0 -1.5708 0 -> xyz=-0.0145 0.0515 -0.0145 rpy=0 -1.57079633 0
- joint left_foot_frame: origin xyz=-0 -0.023 0.042 rpy=-1.5708 -1.5708 0 -> xyz=-0 -0.023 0.042 rpy=-1.57079633 -1.57079633 0
- joint left_hip_pitch: limit lower=-1.5708 upper=1.5708 effort=10 velocity=10 -> lower=-1.5708 upper=1.5708 effort=0.6 velocity=6.6; origin xyz=-0.0145 -0 0.0385 rpy=0 -1.5708 0 -> xyz=-0.0145 0 0.0385 rpy=0 -1.57079633 0
- joint left_hip_roll: limit lower=-0.610865 upper=0.610865 effort=10 velocity=10 -> lower=-0.610865 upper=0.610865 effort=0.6 velocity=6.6; origin xyz=0.02 0 -0.0214 rpy=-1.5708 -0 1.5708 -> xyz=0.02 0 -0.0214 rpy=-1.57079633 -0 1.57079633
- joint left_hip_yaw: limit lower=-1.0472 upper=4.18879 effort=10 velocity=10 -> lower=-1.0472 upper=4.18879 effort=0.6 velocity=6.6; origin xyz=-0 0.036 0 rpy=0 -0 -3.14159 -> xyz=0 0.036 0 rpy=0 -0 3.14159265
- joint left_knee: limit lower=-0.785398 upper=2.35619 effort=10 velocity=10 -> lower=-0.785398 upper=2.35619 effort=0.6 velocity=6.6; origin xyz=0.005 0.062 0 rpy=-0 -0 -0 -> xyz=0.005 0.062 0 rpy=0 -0 0
- joint left_shoulder_pitch: limit lower=-3.14159 upper=3.14159 effort=10 velocity=10 -> lower=-3.14159 upper=3.14159 effort=0.6 velocity=6.6; origin xyz=-0 0.0505 0.081 rpy=1.5708 -0 -3.14159 -> xyz=0 0.0505 0.081 rpy=-1.57079633 -1.57079633 0
- joint left_shoulder_roll: limit lower=0 upper=3.14159 effort=10 velocity=10 -> lower=0 upper=3.14159 effort=0.6 velocity=6.6; origin xyz=-0.0145 0 0.0195 rpy=-3.14159 1.5708 0 -> xyz=0 0.0145 0.0195 rpy=-1.57079633 1.57079633 0
- joint right_ankle_pitch: limit lower=-1.5708 upper=0.610865 effort=10 velocity=10 -> lower=-1.5708 upper=0.610865 effort=0.6 velocity=6.6; origin xyz=0.008 -0.0612131 -0 rpy=-0 0 3.14159 -> xyz=0.008 -0.0612131 0 rpy=0 -0 3.14159265
- joint right_ankle_roll: limit lower=-0.610865 upper=0.610865 effort=10 velocity=10 -> lower=-0.610865 upper=0.610865 effort=0.6 velocity=6.6; origin xyz=-0.0385 0 -0.0145 rpy=3.14159 -1.5708 0 -> xyz=-0.0385 0 -0.0145 rpy=-3.14159265 -1.57079633 0
- joint right_elbow: limit lower=-2.18166 upper=2.18166 effort=10 velocity=10 -> lower=-2.18166 upper=2.18166 effort=0.6 velocity=6.6; origin xyz=-0.0145 -0.0515 -0.0145 rpy=-0 1.5708 0 -> xyz=-0.0145 -0.0515 -0.0145 rpy=-0 1.57079633 0
- joint right_foot_frame: origin xyz=-0 -0.023 0.042 rpy=-1.5708 -1.5708 0 -> xyz=-0 -0.023 0.042 rpy=-1.57079633 -1.57079633 0
- joint right_hip_pitch: limit lower=-1.5708 upper=1.5708 effort=10 velocity=10 -> lower=-1.5708 upper=1.5708 effort=0.6 velocity=6.6; origin xyz=-0.0145 -0 0.0385 rpy=3.14159 1.5708 0 -> xyz=-0.0145 0 0.0385 rpy=3.14159265 1.57079633 0
- joint right_hip_roll: limit lower=-0.610865 upper=0.610865 effort=10 velocity=10 -> lower=-0.610865 upper=0.610865 effort=0.6 velocity=6.6; origin xyz=-0.02 0 -0.0214 rpy=-1.5708 -0 -1.5708 -> xyz=-0.02 0 -0.0214 rpy=-1.57079633 -0 -1.57079633
- joint right_hip_yaw: limit lower=-4.18879 upper=1.0472 effort=10 velocity=10 -> lower=-4.18879 upper=1.0472 effort=0.6 velocity=6.6; origin xyz=0 -0.036 0 rpy=-0 0 0 -> xyz=0 -0.036 0 rpy=0 -0 0
- joint right_knee: limit lower=-0.785398 upper=2.35619 effort=10 velocity=10 -> lower=-0.785398 upper=2.35619 effort=0.6 velocity=6.6; origin xyz=-0.005 -0.062 -0 rpy=-0 0 -0 -> xyz=-0.005 -0.062 0 rpy=0 -0 0
- joint right_shoulder_pitch: limit lower=-3.14159 upper=3.14159 effort=10 velocity=10 -> lower=-3.14159 upper=3.14159 effort=0.6 velocity=6.6; origin xyz=0 -0.0505 0.081 rpy=-1.5708 0 0 -> xyz=0 -0.0505 0.081 rpy=-1.57079633 1.57079633 0
- joint right_shoulder_roll: limit lower=-3.14159 upper=0 effort=10 velocity=10 -> lower=-3.14159 upper=0 effort=0.6 velocity=6.6; origin xyz=0.0145 0 -0.0195 rpy=-3.14159 -1.5708 0 -> xyz=0 -0.0145 -0.0195 rpy=1.57079633 -1.57079633 0
